File: T32 ref.sch (KiCad schematic (older format))
At the start: 89 parts, among them K1 MK20DX256VLH7, K2 MKL04Z32VLC4, T1 MCP1825S, X1 MINI-USB

Commit message: Convert to new library format and fix DRC errors
Parts:
- R7: footprint SOT-23 -> T32 ref:SOT-23
- T1: footprint SOT-223 -> T32 ref:SOT-223
Changed lines of the file:
@@
 EESchema Schematic File Version 2
 LIBS:T32 ref
+LIBS:T32 ref-cache
 EELAYER 25 0
 EELAYER END
@@
 F 0 "R7" H 2530 4130 70  0000 R TNN
 F 1 "~" H 2770 4000 50  0000 L BNN
-F 2 "SOT-23" H 2640 3840 65  0001 L TNN
+F 2 "T32 ref:SOT-23" H 2640 3840 65  0001 L TNN
 F 3 "" H 2650 4050 60  0001 C CNN
 	1    2650 4050
@@
 F 0 "T1" H 3500 1340 70  0000 L BNN
 F 1 "MCP1825S" H 3500 1270 50  0000 L BNN
-F 2 "SOT-223" H 3690 940 65  0001 L TNN
+F 2 "T32 ref:SOT-223" H 3690 940 65  0001 L TNN
 F 3 "" H 3700 1150 60  0001 C CNN
 	1    3700 1150
@@
 	3600 5600 3850 5600
 Wire Wire Line
-	3850 6800 3850 5600
+	3850 5600 3850 6800
 Wire Wire Line
 	3850 5800 4750 5800
@@
 	3700 5500 3700 5600
 Wire Wire Line
-	1100 6800 3850 6800
+	3850 6800 1100 6800
 Wire Wire Line
 	1450 4900 1450 6800
@@
 	3800 2700 2450 2700
 Wire Wire Line
-	2450 2600 2450 2700
-Wire Wire Line
-	1100 2600 2450 2600
+	2450 2700 2450 2600
+Wire Wire Line
+	2450 2600 1100 2600
 Connection ~ 3800 2800
 Wire Wire Line
@@
 	7100 1400 6950 1400
 Wire Wire Line
-	6950 800  6950 1400
+	6950 1400 6950 800
 Wire Wire Line
 	3400 1150 3350 1150
@@
 	3350 1150 3350 800
 Wire Wire Line
-	2450 800  6950 800
+	6950 800  2450 800
 Wire Wire Line
 	3100 900  3100 800

Commit message: Replace common footprints with KiCad versions
Parts:
- C1, C10, C11, C12, C4, C5, C7, C8, C9: footprint T32 ref:C0603 -> Capacitors_SMD:C_0603
- C2, C3, C6: footprint T32 ref:C0805 -> Capacitors_SMD:C_0805
- P1: footprint T32 ref:LED-0805 -> LEDs:LED_0805
- R1: footprint T32 ref:F0805 -> Resistors_SMD:R_0805
- R2, R4: footprint T32 ref:L0603 -> Resistors_SMD:R_0603
- R3, R5, R6, R8: footprint T32 ref:R0603 -> Resistors_SMD:R_0603
- R7: footprint T32 ref:SOT-23 -> TO_SOT_Packages_SMD:SOT-23
- T1: footprint T32 ref:SOT-223 -> TO_SOT_Packages_SMD:SOT-223
Changed lines of the file:
@@
 F 0 "C1" H 3160 970 70  0000 L BNN
 F 1 "0.1uF" H 3159 900 50  0000 L BNN
-F 2 "T32 ref:C0603" H 3090 790 65  0001 L TNN
+F 2 "Capacitors_SMD:C_0603" H 3090 790 65  0001 L TNN
 F 3 "" H 3100 1000 60  0001 C CNN
 	1    3100 1000
@@
 F 0 "C2" H 4210 1270 70  0000 L BNN
 F 1 "2.2uF" H 4209 1200 50  0000 L BNN
-F 2 "T32 ref:C0805" H 4140 1090 65  0001 L TNN
+F 2 "Capacitors_SMD:C_0805" H 4140 1090 65  0001 L TNN
 F 3 "" H 4150 1300 60  0001 C CNN
 	1    4150 1300
@@
 F 0 "C3" H 1310 1520 70  0000 L BNN
 F 1 "2.2uF" H 1309 1450 50  0000 L BNN
-F 2 "T32 ref:C0805" H 1240 1340 65  0001 L TNN
+F 2 "Capacitors_SMD:C_0805" H 1240 1340 65  0001 L TNN
 F 3 "" H 1250 1550 60  0001 C CNN
 	1    1250 1550
@@
 F 0 "C4" H 3860 1920 70  0000 L BNN
 F 1 "0.1uF" H 3859 1850 50  0000 L BNN
-F 2 "T32 ref:C0603" H 3790 1740 65  0001 L TNN
+F 2 "Capacitors_SMD:C_0603" H 3790 1740 65  0001 L TNN
 F 3 "" H 3800 1950 60  0001 C CNN
 	1    3800 1950
@@
 F 0 "C5" H 4210 1920 70  0000 L BNN
 F 1 "0.1uF" H 4209 1850 50  0000 L BNN
-F 2 "T32 ref:C0603" H 4140 1740 65  0001 L TNN
+F 2 "Capacitors_SMD:C_0603" H 4140 1740 65  0001 L TNN
 F 3 "" H 4150 1950 60  0001 C CNN
 	1    4150 1950
@@
 F 0 "C6" H 3160 2870 70  0000 L BNN
 F 1 "2.2uF" H 3159 2800 50  0000 L BNN
-F 2 "T32 ref:C0805" H 3090 2690 65  0001 L TNN
+F 2 "Capacitors_SMD:C_0805" H 3090 2690 65  0001 L TNN
 F 3 "" H 3100 2900 60  0001 C CNN
 	1    3100 2900
@@
 F 0 "C7" H 3860 3020 70  0000 L BNN
 F 1 "0.1uF" H 3859 2950 50  0000 L BNN
-F 2 "T32 ref:C0603" H 3790 2840 65  0001 L TNN
+F 2 "Capacitors_SMD:C_0603" H 3790 2840 65  0001 L TNN
 F 3 "" H 3800 3050 60  0001 C CNN
 	1    3800 3050
@@
 F 0 "C8" H 4210 3020 70  0000 L BNN
 F 1 "0.1uF" H 4209 2950 50  0000 L BNN
-F 2 "T32 ref:C0603" H 4140 2840 65  0001 L TNN
+F 2 "Capacitors_SMD:C_0603" H 4140 2840 65  0001 L TNN
 F 3 "" H 4150 3050 60  0001 C CNN
 	1    4150 3050
@@
 F 0 "C9" H 2710 4270 70  0000 L BNN
 F 1 "0.1uF" H 2709 4200 50  0000 L BNN
-F 2 "T32 ref:C0603" H 2640 4090 65  0001 L TNN
+F 2 "Capacitors_SMD:C_0603" H 2640 4090 65  0001 L TNN
 F 3 "" H 2650 4300 60  0001 C CNN
 	1    2650 4300
@@
 F 0 "C10" H 3410 4270 70  0000 L BNN
 F 1 "22pF" H 3409 4200 50  0000 L BNN
-F 2 "T32 ref:C0603" H 3340 4090 65  0001 L TNN
+F 2 "Capacitors_SMD:C_0603" H 3340 4090 65  0001 L TNN
 F 3 "" H 3350 4300 60  0001 C CNN
 	1    3350 4300
@@
 F 0 "C11" H 3760 4270 70  0000 L BNN
 F 1 "22pF" H 3759 4200 50  0000 L BNN
-F 2 "T32 ref:C0603" H 3690 4090 65  0001 L TNN
+F 2 "Capacitors_SMD:C_0603" H 3690 4090 65  0001 L TNN
 F 3 "" H 3700 4300 60  0001 C CNN
 	1    3700 4300
@@
 F 0 "C12" H 2160 5320 70  0000 L BNN
 F 1 "0.1uF" H 2159 5250 50  0000 L BNN
-F 2 "T32 ref:C0603" H 2090 5140 65  0001 L TNN
+F 2 "Capacitors_SMD:C_0603" H 2090 5140 65  0001 L TNN
 F 3 "" H 2100 5350 60  0001 C CNN
 	1    2100 5350
@@
 F 0 "P1" H 7090 6840 70  0000 L BNN
 F 1 "~" H 6940 6740 65  0001 L TNN
-F 2 "T32 ref:LED-0805" H 6940 6640 65  0001 L TNN
+F 2 "LEDs:LED_0805" H 6940 6640 65  0001 L TNN
 F 3 "" H 6950 6850 60  0001 C CNN
 	1    6950 6850
@@
 F 0 "R1" V 1470 1040 70  0000 R TNN
 F 1 "FUSE" V 1400 1040 50  0000 R TNN
-F 2 "T32 ref:F0805" H 1490 890 65  0001 L TNN
+F 2 "Resistors_SMD:R_0805" H 1490 890 65  0001 L TNN
 F 3 "" H 1500 1100 60  0001 C CNN
 	1    1500 1100
@@
 F 0 "R2" V 3070 2080 70  0000 R TNN
 F 1 "~" H 3000 2000 50  0000 L BNN
-F 2 "T32 ref:L0603" H 3090 1890 65  0001 L TNN
+F 2 "Resistors_SMD:R_0603" H 3090 1890 65  0001 L TNN
 F 3 "" H 3100 2100 60  0001 C CNN
 	1    3100 2100
@@
 F 0 "R3" H 3430 2681 70  0000 L BNN
 F 1 "470R" H 3589 2680 50  0000 L BNN
-F 2 "T32 ref:R0603" H 3540 2590 65  0001 L TNN
+F 2 "Resistors_SMD:R_0603" H 3540 2590 65  0001 L TNN
 F 3 "" H 3550 2800 60  0001 C CNN
 	1    3550 2800
@@
 F 0 "R4" H 2650 3100 70  0000 L BNN
 F 1 "~" H 2740 3090 65  0001 L TNN
-F 2 "T32 ref:L0603" H 2740 2990 65  0001 L TNN
+F 2 "Resistors_SMD:R_0603" H 2740 2990 65  0001 L TNN
 F 3 "" H 2750 3200 60  0001 C CNN
 	1    2750 3200
@@
 F 0 "R5" H 3430 3281 70  0000 L BNN
 F 1 "33R" H 3589 3280 50  0000 L BNN
-F 2 "T32 ref:R0603" H 3540 3190 65  0001 L TNN
+F 2 "Resistors_SMD:R_0603" H 3540 3190 65  0001 L TNN
 F 3 "" H 3550 3400 60  0001 C CNN
 	1    3550 3400
@@
 F 0 "R6" H 3430 3481 70  0000 L BNN
 F 1 "33R" H 3589 3480 50  0000 L BNN
-F 2 "T32 ref:R0603" H 3540 3390 65  0001 L TNN
+F 2 "Resistors_SMD:R_0603" H 3540 3390 65  0001 L TNN
 F 3 "" H 3550 3600 60  0001 C CNN
 	1    3550 3600
@@
 F 0 "R7" H 2530 4130 70  0000 R TNN
 F 1 "~" H 2770 4000 50  0000 L BNN
-F 2 "T32 ref:SOT-23" H 2640 3840 65  0001 L TNN
+F 2 "TO_SOT_Packages_SMD:SOT-23" H 2640 3840 65  0001 L TNN
 F 3 "" H 2650 4050 60  0001 C CNN
 	1    2650 4050
@@
 F 0 "R8" V 6910 7150 70  0000 R TNN
 F 1 "470R" V 6840 7150 50  0000 R TNN
-F 2 "T32 ref:R0603" H 6940 6990 65  0001 L TNN
+F 2 "Resistors_SMD:R_0603" H 6940 6990 65  0001 L TNN
 F 3 "" H 6950 7200 60  0001 C CNN
 	1    6950 7200
@@
 F 0 "T1" H 3500 1340 70  0000 L BNN
 F 1 "MCP1825S" H 3500 1270 50  0000 L BNN
-F 2 "T32 ref:SOT-223" H 3690 940 65  0001 L TNN
+F 2 "TO_SOT_Packages_SMD:SOT-223" H 3690 940 65  0001 L TNN
 F 3 "" H 3700 1150 60  0001 C CNN
 	1    3700 1150

Commit message: Add part numbers to schematic and export BOM
Parts:
- C1, C12, C4, C5, C7, C8, C9: Mfg_Part_No (none) -> GRM155R71A104KA01D
- C10, C11: Mfg_Part_No (none) -> VJ0603A220JXACW1BC
- C2, C3, C6: Mfg_Part_No (none) -> TMK212B7225KG-TR
- G1: Mfg_Part_No (none) -> ABL-16.000MHz-B1U
- G2: Mfg_Part_No (none) -> CFS206-32.768KDZF-UB
- K1: Mfg_Part_No (none) -> MK20DX256VLH7
- P1: Mfg_Part_No (none) -> SML-211DTT86
- R1: Mfg_Part_No (none) -> 0ZCK0050FF2E
- R2, R4: Mfg_Part_No (none) -> BLM18AG601SN1D
- R3, R8: Mfg_Part_No (none) -> CRCW0603470RFKEA
- R5, R6: Mfg_Part_No (none) -> ERJ-PA3F33R0V
- R7: Mfg_Part_No (none) -> BAT54C,215
- S1: Mfg_Part_No (none) -> SKHHPKA010
- T1: Mfg_Part_No (none) -> MCP1825S-3302E/DB
- X1: Mfg_Part_No (none) -> 67503-1020
Changed lines of the file:
@@
 EESchema Schematic File Version 2
 LIBS:T32 ref
-LIBS:T32 ref-cache
 EELAYER 25 0
 EELAYER END
@@
 F 2 "Capacitors_SMD:C_0603" H 3090 790 65  0001 L TNN
 F 3 "" H 3100 1000 60  0001 C CNN
+F 4 "GRM155R71A104KA01D" H 3100 1000 60  0001 C CNN "Mfg_Part_No"
 	1    3100 1000
 	1    0    0    -1
@@
 F 2 "Capacitors_SMD:C_0805" H 4140 1090 65  0001 L TNN
 F 3 "" H 4150 1300 60  0001 C CNN
+F 4 "TMK212B7225KG-TR" H 4150 1300 60  0001 C CNN "Mfg_Part_No"
 	1    4150 1300
 	1    0    0    -1
@@
 F 2 "Capacitors_SMD:C_0805" H 1240 1340 65  0001 L TNN
 F 3 "" H 1250 1550 60  0001 C CNN
+F 4 "TMK212B7225KG-TR" H 1250 1550 60  0001 C CNN "Mfg_Part_No"
 	1    1250 1550
 	1    0    0    -1
@@
 F 2 "Capacitors_SMD:C_0603" H 3790 1740 65  0001 L TNN
 F 3 "" H 3800 1950 60  0001 C CNN
+F 4 "GRM155R71A104KA01D" H 3800 1950 60  0001 C CNN "Mfg_Part_No"
 	1    3800 1950
 	1    0    0    -1
@@
 F 2 "Capacitors_SMD:C_0603" H 4140 1740 65  0001 L TNN
 F 3 "" H 4150 1950 60  0001 C CNN
+F 4 "GRM155R71A104KA01D" H 4150 1950 60  0001 C CNN "Mfg_Part_No"
 	1    4150 1950
 	1    0    0    -1
@@
 F 2 "Capacitors_SMD:C_0805" H 3090 2690 65  0001 L TNN
 F 3 "" H 3100 2900 60  0001 C CNN
+F 4 "TMK212B7225KG-TR" H 3100 2900 60  0001 C CNN "Mfg_Part_No"
 	1    3100 2900
 	1    0    0    -1
@@
 F 2 "Capacitors_SMD:C_0603" H 3790 2840 65  0001 L TNN
 F 3 "" H 3800 3050 60  0001 C CNN
+F 4 "GRM155R71A104KA01D" H 3800 3050 60  0001 C CNN "Mfg_Part_No"
 	1    3800 3050
 	1    0    0    -1
@@
 F 2 "Capacitors_SMD:C_0603" H 4140 2840 65  0001 L TNN
 F 3 "" H 4150 3050 60  0001 C CNN
+F 4 "GRM155R71A104KA01D" H 4150 3050 60  0001 C CNN "Mfg_Part_No"
 	1    4150 3050
 	1    0    0    -1
@@
 F 2 "Capacitors_SMD:C_0603" H 2640 4090 65  0001 L TNN
 F 3 "" H 2650 4300 60  0001 C CNN
+F 4 "GRM155R71A104KA01D" H 2650 4300 60  0001 C CNN "Mfg_Part_No"
 	1    2650 4300
 	1    0    0    -1
@@
 F 2 "Capacitors_SMD:C_0603" H 3340 4090 65  0001 L TNN
 F 3 "" H 3350 4300 60  0001 C CNN
+F 4 "VJ0603A220JXACW1BC" H 3350 4300 60  0001 C CNN "Mfg_Part_No"
 	1    3350 4300
 	1    0    0    -1
@@
 F 2 "Capacitors_SMD:C_0603" H 3690 4090 65  0001 L TNN
 F 3 "" H 3700 4300 60  0001 C CNN
+F 4 "VJ0603A220JXACW1BC" H 3700 4300 60  0001 C CNN "Mfg_Part_No"
 	1    3700 4300
 	1    0    0    -1
@@
 F 2 "Capacitors_SMD:C_0603" H 2090 5140 65  0001 L TNN
 F 3 "" H 2100 5350 60  0001 C CNN
+F 4 "GRM155R71A104KA01D" H 2100 5350 60  0001 C CNN "Mfg_Part_No"
 	1    2100 5350
 	1    0    0    -1
@@
 F 2 "T32 ref:HC49US" H 4040 3740 65  0001 L TNN
 F 3 "" H 4050 3950 60  0001 C CNN
+F 4 "ABL-16.000MHz-B1U" H 4050 3950 60  0001 C CNN "Mfg_Part_No"
 	1    4050 3950
 	0    1    1    0
@@
 F 2 "T32 ref:TC26H" H 4040 4140 65  0001 L TNN
 F 3 "" H 4050 4350 60  0001 C CNN
+F 4 "CFS206-32.768KDZF-UB" H 4050 4350 60  0001 C CNN "Mfg_Part_No"
 	1    4050 4350
 	0    1    1    0
@@
 F 2 "T32 ref:LQFP64-05" H 5540 3790 65  0001 L TNN
 F 3 "" H 5550 4000 60  0001 C CNN
+F 4 "MK20DX256VLH7" H 5550 4000 60  0001 C CNN "Mfg_Part_No"
 	1    5550 4000
 	1    0    0    -1
@@
 F 2 "LEDs:LED_0805" H 6940 6640 65  0001 L TNN
 F 3 "" H 6950 6850 60  0001 C CNN
+F 4 "SML-211DTT86" H 6950 6850 60  0001 C CNN "Mfg_Part_No"
 	1    6950 6850
 	1    0    0    -1
@@
 F 2 "Resistors_SMD:R_0805" H 1490 890 65  0001 L TNN
 F 3 "" H 1500 1100 60  0001 C CNN
+F 4 "0ZCK0050FF2E" H 1500 1100 60  0001 C CNN "Mfg_Part_No"
 	1    1500 1100
 	0    -1   -1   0
@@
 F 2 "Resistors_SMD:R_0603" H 3090 1890 65  0001 L TNN
 F 3 "" H 3100 2100 60  0001 C CNN
+F 4 "BLM18AG601SN1D" H 3100 2100 60  0001 C CNN "Mfg_Part_No"
 	1    3100 2100
 	0    -1   -1   0
@@
 F 2 "Resistors_SMD:R_0603" H 3540 2590 65  0001 L TNN
 F 3 "" H 3550 2800 60  0001 C CNN
+F 4 "CRCW0603470RFKEA" H 3550 2800 60  0001 C CNN "Mfg_Part_No"
 	1    3550 2800
 	1    0    0    -1
@@
 F 2 "Resistors_SMD:R_0603" H 2740 2990 65  0001 L TNN
 F 3 "" H 2750 3200 60  0001 C CNN
+F 4 "BLM18AG601SN1D" H 2750 3200 60  0001 C CNN "Mfg_Part_No"
 	1    2750 3200
 	1    0    0    -1
@@
 F 2 "Resistors_SMD:R_0603" H 3540 3190 65  0001 L TNN
 F 3 "" H 3550 3400 60  0001 C CNN
+F 4 "ERJ-PA3F33R0V" H 3550 3400 60  0001 C CNN "Mfg_Part_No"
 	1    3550 3400
 	1    0    0    -1
@@
 F 2 "Resistors_SMD:R_0603" H 3540 3390 65  0001 L TNN
 F 3 "" H 3550 3600 60  0001 C CNN
+F 4 "ERJ-PA3F33R0V" H 3550 3600 60  0001 C CNN "Mfg_Part_No"
 	1    3550 3600
 	1    0    0    -1
@@
 F 2 "TO_SOT_Packages_SMD:SOT-23" H 2640 3840 65  0001 L TNN
 F 3 "" H 2650 4050 60  0001 C CNN
+F 4 "BAT54C,215" H 2650 4050 60  0001 C CNN "Mfg_Part_No"
 	1    2650 4050
 	-1   0    0    -1
@@
 F 2 "Resistors_SMD:R_0603" H 6940 6990 65  0001 L TNN
 F 3 "" H 6950 7200 60  0001 C CNN
+F 4 "CRCW0603470RFKEA" H 6950 7200 60  0001 C CNN "Mfg_Part_No"
 	1    6950 7200
 	0    -1   -1   0
@@
 F 2 "T32 ref:ALPS_SKHH" H 1640 5940 65  0001 L TNN
 F 3 "" H 1650 6150 60  0001 C CNN
+F 4 "SKHHPKA010" H 1650 6150 60  0001 C CNN "Mfg_Part_No"
 	1    1650 6150
 	1    0    0    -1
@@
 F 2 "TO_SOT_Packages_SMD:SOT-223" H 3690 940 65  0001 L TNN
 F 3 "" H 3700 1150 60  0001 C CNN
+F 4 "MCP1825S-3302E/DB" H 3700 1150 60  0001 C CNN "Mfg_Part_No"
 	1    3700 1150
 	1    0    0    -1
@@
 F 2 "T32 ref:MOLEX_SD-67503-010" H 740 3390 65  0001 L TNN
 F 3 "" H 750 3600 60  0001 C CNN
+F 4 "67503-1020" H 750 3600 60  0001 C CNN "Mfg_Part_No"
 	1    750  3600
 	1    0    0    -1
