File: T32_ref.sch (KiCad schematic (older format))
At the start: 89 parts, among them K1 MK20DX256VLH7, K2 MKL04Z32VLC4, T1 MCP1825S, X1 MINI-USB

Commit message: Fix cap footprint
Fixes #2
Parts:
- C1, C12, C4, C5, C7, C8, C9: symbol CAPACITOR-0.1UF -> T32_ref:CAPACITOR-0.1UF
- C10, C11: symbol CAPACITOR-22PF -> T32_ref:CAPACITOR-22PF
- C2, C3, C6: symbol CAPACITOR-2.2UF -> T32_ref:CAPACITOR-2.2UF
- G1: symbol CRYSTAL-HC49US -> T32_ref:CRYSTAL-HC49US
- G2: symbol CRYSTAL-TC26H -> T32_ref:CRYSTAL-TC26H
- K1: symbol MK20DX256VLH7 -> T32_ref:MK20DX256VLH7
- K2: symbol MKL04Z32VLC4 -> T32_ref:MKL04Z32VLC4
- P1: symbol LED -> T32_ref:LED
- R1: symbol FUSE -> T32_ref:FUSE
- R2, R4: symbol FERRITE -> T32_ref:FERRITE
- R3, R8: symbol RESISTOR-470R -> T32_ref:RESISTOR-470R
- R5, R6: symbol RESISTOR-33R -> T32_ref:RESISTOR-33R
- R7: symbol DIODE_DUAL -> T32_ref:DIODE_DUAL
- S1: symbol TACT_SWITCH -> T32_ref:TACT_SWITCH
- SJ1: symbol SOLDERJUMPER -> T32_ref:SOLDERJUMPER
- SX1, SX10, SX11, SX12, SX13, SX14, SX15, SX16, SX17, SX18, SX19, SX2, SX20, SX21, SX22, SX23, SX24, SX25, SX26, SX27, SX28, SX29, SX3, SX30, SX31, SX32, SX33, SX34, SX35, SX36, SX37, SX38, SX39, SX4, SX40, SX41, SX42, SX43, SX44, SX45, SX46, SX47, SX48, SX49, SX5, SX50, SX51, SX52, SX53, SX54, SX55, SX56, SX57, SX58, SX59, SX6, SX60, SX7, SX8, SX9: symbol PIN -> T32_ref:PIN
- T1: symbol LDO -> T32_ref:LDO
- X1: symbol MINI-USBMOLEX_0675031230 -> T32_ref:MINI-USBMOLEX_0675031230
